File: mibo48_stm32f303/mibo48_stm32f303.sch (KiCad schematic (older format))
At the start: 30 parts, among them J1 Conn_01x02, J2 Conn_01x22, J3 Conn_01x22, J4 USB_B_Micro, J5 Conn_01x04, SW1 Reset, U1 STM32F303CBTx, U2 AMS1117-3.3, Y1 8MHz

Commit message: - fully routed, only labelling is missing - kicad 5 project with new libraries and footprints
Parts:
- added C10, C9: 22pF, Capacitor_SMD:C_0603_1608Metric, symbol Device:C
- added Y2: 32.768kHz, Crystal:Crystal_C26-LF_D2.1mm_L6.5mm_Horizontal, symbol Device:Crystal
- C1, C11, C2, C3, C4, C5, C6, C7, C8: footprint Capacitors_SMD:C_0603 -> Capacitor_SMD:C_0603_1608Metric
- D1, D2: footprint Diodes_SMD:D_0603 -> LED_SMD:LED_0603_1608Metric
- J1: footprint Pin_Headers:Pin_Header_Straight_1x02_Pitch2.54mm -> Connector_PinHeader_2.54mm:PinHeader_1x02_P2.54mm_Vertical
- J2, J3: footprint Pin_Headers:Pin_Header_Straight_1x22_Pitch2.54mm -> Connector_PinHeader_2.54mm:PinHeader_1x22_P2.54mm_Vertical
- J4: footprint Connectors:USB_Micro-B -> Connector_USB:USB_Micro-B_Molex-105017-0001
- J5: footprint Pin_Headers:Pin_Header_Straight_1x04_Pitch2.54mm -> Connector_PinHeader_2.54mm:PinHeader_1x04_P2.54mm_Vertical
- R1, R10, R2, R3, R4, R5, R6, R7, R8, R9: footprint Resistors_SMD:R_0603 -> Resistor_SMD:R_0603_1608Metric
- SW1: footprint Buttons_Switches_SMD:SW_SPST_FSMSM -> Button_Switch_SMD:SW_SPST_CK_RS282G05A3
- U1: footprint Housings_QFP:LQFP-48_7x7mm_Pitch0.5mm -> Package_QFP:LQFP-48_7x7mm_P0.5mm
- U2: footprint TO_SOT_Packages_SMD:SOT-223 -> Package_TO_SOT_SMD:SOT-223
- Y1: footprint Crystals:Crystal_HC49-U_Vertical -> Crystal:Crystal_HC49-4H_Vertical
Connections:
- wire segments 186 -> 196
