File: mibo20_stm32/mibo20_stm32.sch (KiCad schematic (older format))
At the start: 24 parts, among them J1 Conn_01x02, J2 Conn_01x13, J3 Conn_01x13, J4 USB_B_Micro, J5 Conn_01x04, SW1 Reset, U1 STM32F070F6Px, U2 AMS1117-3.3, Y1 8MHz

Commit message: Test commit
Parts:
- removed R8, R9: 22R, Resistor_SMD:R_0603_1608Metric, symbol Device:R
Connections:
- wire segments 118 -> 116
Changed lines of the file:
@@
 Text Label 10200 2400 2    50   ~ 0
 5V
-$Comp
-L Device:R R8
-U 1 1 5BAD065C
-P 9550 3300
-F 0 "R8" V 9343 3300 50  0000 C CNN
-F 1 "22R" V 9450 3300 50  0000 C CNN
-F 2 "Resistor_SMD:R_0603_1608Metric" V 9480 3300 50  0001 C CNN
-F 3 "~" H 9550 3300 50  0001 C CNN
-	1    9550 3300
-	0    -1   1    0
-$EndComp
-$Comp
-L Device:R R9
-U 1 1 5BAD078C
-P 9550 3500
-F 0 "R9" V 9650 3500 50  0000 C CNN
-F 1 "22R" V 9450 3500 50  0000 C CNN
-F 2 "Resistor_SMD:R_0603_1608Metric" V 9480 3500 50  0001 C CNN
-F 3 "~" H 9550 3500 50  0001 C CNN
-	1    9550 3500
-	0    -1   1    0
-$EndComp
 Wire Wire Line
 	10100 3100 10000 3100
@@
 Wire Wire Line
 	9800 3400 9800 3500
-Wire Wire Line
-	9800 3500 9700 3500
-Wire Wire Line
-	9400 3500 9000 3500
-Wire Wire Line
-	9400 3300 9000 3300
 Text Label 9000 3500 0    50   ~ 0
 PA11
@@
 Text Label 5900 2900 2    50   ~ 0
 PA11
-Wire Wire Line
-	9700 3300 10100 3300
 Text Label 3900 3200 0    50   ~ 0
 PB1
@@
 	-1   0    0    -1
 $EndComp
+Wire Wire Line
+	9000 3300 10100 3300
+Wire Wire Line
+	9000 3500 9800 3500
 $EndSCHEMATC

Commit message: V1.0 - Fully routed with description
Parts:
- added C5: 100nF, Capacitor_SMD:C_0603_1608Metric, symbol Device:C
- added C7: 1uF, Capacitor_SMD:C_0603_1608Metric, symbol Device:C
- C3: value 10nF -> 100nF
- C4: value 100nF -> 4.7uF
- C6: renamed from C5; value 100nF -> 10nF
- D2: value GREEN -> RED
- renumbered C11 to C9, R10 to R4
Connections:
- net labels added: PA13, PA14, PF0, PF1
- wire segments 116 -> 119
Other:
- moved on the sheet: U2

Commit message: Q1 and SW1 swapped
Parts:
- added JP1: SolderJumper_2_Open, symbol Jumper:SolderJumper_2_Open
Connections:
- wire segments 119 -> 120
Changed lines of the file:
@@
 Text Label 5800 3150 2    50   ~ 0
 PA7
-Text Label 1550 5700 0    50   ~ 0
+Text Label 1100 5700 0    50   ~ 0
 RESET
 Wire Wire Line
@@
 	1550 5600 1850 5600
 Wire Wire Line
-	1850 5700 1550 5700
-Wire Wire Line
-	1550 5800 1850 5800
-Wire Wire Line
-	1850 5900 1550 5900
-Wire Wire Line
-	1550 6000 1850 6000
-Wire Wire Line
-	1850 6100 1550 6100
-Wire Wire Line
-	1550 6200 1850 6200
+	1150 6000 850  6000
+Wire Wire Line
+	1550 5700 1850 5700
+Wire Wire Line
+	1850 5800 1550 5800
+Wire Wire Line
+	1550 5900 1850 5900
+Wire Wire Line
+	1850 6000 1550 6000
+Wire Wire Line
+	1550 6100 1850 6100
+Wire Wire Line
+	1850 6200 1550 6200
 Wire Wire Line
 	1850 6300 1550 6300
 Wire Wire Line
-	1850 6400 1550 6400
-Wire Wire Line
-	1550 6500 1850 6500
+	1550 6400 1850 6400
 Wire Wire Line
 	1850 6600 1550 6600
@@
 Text Label 7600 4650 2    50   ~ 0
 PA12
+Text Label 1550 5700 0    50   ~ 0
+PA0
 Text Label 1550 5800 0    50   ~ 0
-PA0
+PA1
 Text Label 1550 5900 0    50   ~ 0
-PA1
+PA2
 Text Label 1550 6000 0    50   ~ 0
-PA2
+PA3
 Text Label 1550 6100 0    50   ~ 0
-PA3
+PA4
 Text Label 1550 6200 0    50   ~ 0
-PA4
+PA5
 Text Label 1550 6300 0    50   ~ 0
-PA5
-Text Label 1550 6400 0    50   ~ 0
 PA6
 Text Label 6800 4750 0    50   ~ 0
@@
 Text Label 6800 4850 0    50   ~ 0
 OSC_OUT
-Text Label 1550 6500 0    50   ~ 0
+Text Label 1550 6400 0    50   ~ 0
 PA7
 $Comp
@@
 	2850 6100 3150 6100
 Text Label 3150 6000 2    50   ~ 0
-PB1
+RESET
 Text Label 3150 6100 2    50   ~ 0
 PA9
@@
 PA14
 Connection ~ 2500 1650
+Text Label 1550 6500 0    50   ~ 0
+PB1
+Wire Wire Line
+	1850 6500 1550 6500
+$Comp
+L Jumper:SolderJumper_2_Open JP1
+U 1 1 5BAC57D8
+P 5400 4950
+F 0 "JP1" H 5400 5155 50  0000 C CNN
+F 1 "SolderJumper_2_Open" H 5400 5064 50  0000 C CNN
+F 2 "" H 5400 4950 50  0001 C CNN
+F 3 "~" H 5400 4950 50  0001 C CNN
+	1    5400 4950
+	1    0    0    -1
+$EndComp
 $EndSCHEMATC

Commit message: Jumper for USB added
Parts:
- added JP2: SolderJumper_2_Open, mibo20_stm32:SolderJumper-2_P0.8mm_Open_RoundedPad0.6x0.8mm, symbol Jumper:SolderJumper_2_Open
- JP1: footprint (none) -> mibo20_stm32:SolderJumper-2_P0.8mm_Open_RoundedPad0.6x0.8mm
Connections:
- wire segments 120 -> 125
Changed lines of the file:
@@
 Text Label 5800 3150 2    50   ~ 0
 PA7
-Text Label 1100 5700 0    50   ~ 0
-RESET
 Wire Wire Line
 	1300 1650 1500 1650
@@
 Wire Wire Line
 	9650 4550 9650 4650
-Text Label 8850 4650 0    50   ~ 0
+Text Label 7900 4650 0    50   ~ 0
 PA11
-Text Label 8850 4550 0    50   ~ 0
+Text Label 7900 4550 0    50   ~ 0
 PA12
-Text Notes 7450 4000 2    50   ~ 0
+Text Notes 7050 4000 2    50   ~ 0
 Shared functions
 Wire Wire Line
-	6800 4250 7600 4250
-Wire Wire Line
-	6800 4350 7600 4350
-Text Label 6800 4250 0    50   ~ 0
+	6400 4250 7200 4250
+Wire Wire Line
+	6400 4350 7200 4350
+Text Label 6400 4250 0    50   ~ 0
 PA12
-Text Label 6800 4350 0    50   ~ 0
+Text Label 6400 4350 0    50   ~ 0
 PA11
-Text Label 7600 4250 2    50   ~ 0
+Text Label 7200 4250 2    50   ~ 0
 USB_D+
-Text Label 7600 4350 2    50   ~ 0
+Text Label 7200 4350 2    50   ~ 0
 USB_D-
 Text Label 3600 4650 2    50   ~ 0
 LED1
-Text Label 7600 4450 2    50   ~ 0
+Text Label 7200 4450 2    50   ~ 0
 LED1
 Wire Wire Line
-	7600 4450 6800 4450
-Wire Wire Line
-	7600 4550 6800 4550
+	7200 4450 6400 4450
+Wire Wire Line
+	7200 4550 6400 4550
 $Comp
 L Connector_Generic:Conn_01x04 J5
@@
 	1550 5600 1850 5600
 Wire Wire Line
-	1150 6000 850  6000
-Wire Wire Line
 	1550 5700 1850 5700
 Wire Wire Line
@@
 Text Label 3900 3550 0    50   ~ 0
 PB1
-Text Label 6800 4450 0    50   ~ 0
+Text Label 6400 4450 0    50   ~ 0
 PB1
-Text Label 6800 4550 0    50   ~ 0
+Text Label 6400 4550 0    50   ~ 0
 PA9
-Text Label 6800 4650 0    50   ~ 0
+Text Label 6400 4650 0    50   ~ 0
 PA10
-Text Label 7600 4550 2    50   ~ 0
+Text Label 7200 4550 2    50   ~ 0
 PA11
-Text Label 7600 4650 2    50   ~ 0
+Text Label 7200 4650 2    50   ~ 0
 PA12
 Text Label 1550 5700 0    50   ~ 0
@@
 Text Label 1550 6300 0    50   ~ 0
 PA6
-Text Label 6800 4750 0    50   ~ 0
+Text Label 6400 4750 0    50   ~ 0
 OSC_IN
-Text Label 6800 4850 0    50   ~ 0
+Text Label 6400 4850 0    50   ~ 0
 OSC_OUT
 Text Label 1550 6400 0    50   ~ 0
@@
 Connection ~ 2500 2050
 Wire Wire Line
-	7600 4750 6800 4750
-Wire Wire Line
-	6800 4850 7600 4850
-Text Label 7600 4750 2    50   ~ 0
+	7200 4750 6400 4750
+Wire Wire Line
+	6400 4850 7200 4850
+Text Label 7200 4750 2    50   ~ 0
 PF0
-Text Label 7600 4850 2    50   ~ 0
+Text Label 7200 4850 2    50   ~ 0
 PF1
 Wire Wire Line
@@
 	5400 1750 5650 1750
 Connection ~ 5400 1750
-Wire Wire Line
-	8850 4550 9150 4550
-Wire Wire Line
-	8850 4650 9150 4650
-Wire Wire Line
-	9150 4350 8850 4350
-Text Label 8850 4350 0    50   ~ 0
+Text Label 7900 4350 0    50   ~ 0
 5V
 Wire Wire Line
@@
 	5900 3550 5400 3550
 Wire Wire Line
-	6800 4650 7600 4650
-Text Label 6800 4950 0    50   ~ 0
+	6400 4650 7200 4650
+Text Label 6400 4950 0    50   ~ 0
 SWDIO
-Text Label 6800 5050 0    50   ~ 0
+Text Label 6400 5050 0    50   ~ 0
 SWDCLK
 Wire Wire Line
-	7600 4950 6800 4950
-Wire Wire Line
-	6800 5050 7600 5050
-Text Label 7600 4950 2    50   ~ 0
+	7200 4950 6400 4950
+Wire Wire Line
+	6400 5050 7200 5050
+Text Label 7200 4950 2    50   ~ 0
 PA13
-Text Label 7600 5050 2    50   ~ 0
+Text Label 7200 5050 2    50   ~ 0
 PA14
 Connection ~ 2500 1650
@@
 L Jumper:SolderJumper_2_Open JP1
 U 1 1 5BAC57D8
-P 5400 4950
-F 0 "JP1" H 5400 5155 50  0000 C CNN
-F 1 "SolderJumper_2_Open" H 5400 5064 50  0000 C CNN
-F 2 "" H 5400 4950 50  0001 C CNN
-F 3 "~" H 5400 4950 50  0001 C CNN
-	1    5400 4950
-	1    0    0    -1
-$EndComp
+P 8700 4550
+F 0 "JP1" H 8700 4648 50  0000 C CNN
+F 1 "SolderJumper_2_Open" H 8700 4664 50  0001 C CNN
+F 2 "mibo20_stm32:SolderJumper-2_P0.8mm_Open_RoundedPad0.6x0.8mm" H 8700 4550 50  0001 C CNN
+F 3 "~" H 8700 4550 50  0001 C CNN
+	1    8700 4550
+	1    0    0    -1
+$EndComp
+$Comp
+L Jumper:SolderJumper_2_Open JP2
+U 1 1 5BB2DDDE
+P 8700 4800
+F 0 "JP2" H 8700 4898 50  0000 C CNN
+F 1 "SolderJumper_2_Open" H 8700 4914 50  0001 C CNN
+F 2 "mibo20_stm32:SolderJumper-2_P0.8mm_Open_RoundedPad0.6x0.8mm" H 8700 4800 50  0001 C CNN
+F 3 "~" H 8700 4800 50  0001 C CNN
+	1    8700 4800
+	1    0    0    -1
+$EndComp
+Wire Wire Line
+	9150 4550 8850 4550
+Wire Wire Line
+	9150 4650 9050 4650
+Wire Wire Line
+	9050 4650 9050 4800
+Wire Wire Line
+	9050 4800 8850 4800
+Wire Wire Line
+	7900 4550 8550 4550
+Wire Wire Line
+	8550 4800 8400 4800
+Wire Wire Line
+	8400 4800 8400 4650
+Wire Wire Line
+	7900 4650 8400 4650
+Wire Wire Line
+	7900 4350 9150 4350
 $EndSCHEMATC
