File: mibo100_imxrt/mibo100_imxrt.sch (KiCad schematic (older format))
At the start: 23 parts, among them J4 USB_B_Micro, J5 Conn_01x04, U2 AMS1117-3.3, Y1 8MHz, Y2 32.768kHz

Commit message: some progress with the imxrt
Parts:
- removed C10: 22pF, Capacitor_SMD:C_0603_1608Metric, symbol Device:C
- removed C8: 4.7uF, Capacitor_SMD:C_0603_1608Metric, symbol Device:C
- removed J5: Conn_01x04, Connector_PinHeader_2.54mm:PinHeader_1x04_P2.54mm_Vertical, symbol Connector_Generic:Conn_01x04
- removed U2: AMS1117-3.3, Package_TO_SOT_SMD:SOT-223, symbol Regulator_Linear:AMS1117-3.3
- removed Y1: 8MHz, Crystal:Crystal_HC49-4H_Vertical, symbol Device:Crystal
- removed Y2: 32.768kHz, Crystal:Crystal_C26-LF_D2.1mm_L6.5mm_Horizontal, symbol Device:Crystal
- added C1, C13, C18, C20, C21, C22, C25, C26, C27, C5, C6: 220nF, Capacitor_SMD:C_0402_1005Metric, symbol Device:C
- added C15, C17, C24, C28: 4.7uF, Capacitor_SMD:C_0603_1608Metric, symbol Device:C
- added C16, C19, C29: 100nF, Capacitor_SMD:C_0603_1608Metric, symbol Device:C
- added C23: 33uF, Capacitor_SMD:C_0603_1608Metric, symbol Device:C
- added C4: 10uF, Capacitor_SMD:C_0603_1608Metric, symbol Device:C
- added J1, J2: Conn_01x26, Connector_PinHeader_2.54mm:PinHeader_1x26_P2.54mm_Vertical, symbol Connector_Generic:Conn_01x26
- added J3: Conn_02x02_Odd_Even, Connector_PinHeader_2.54mm:PinHeader_2x02_P2.54mm_Vertical, symbol Connector_Generic:Conn_02x02_Odd_Even
- added J5: Conn_01x05, Connector_PinHeader_2.54mm:PinHeader_1x05_P2.54mm_Vertical, symbol Connector_Generic:Conn_01x05
- added L1: 47nH, Inductor_SMD:L_0805_2012Metric, symbol Device:L
- added L2: 2.2 uH, Inductor_SMD:L_1210_3225Metric_Pad1.42x2.65mm_HandSolder, symbol Device:L_Core_Ferrite
- added L3: 4.7 uH, Inductor_SMD:L_1210_3225Metric_Pad1.42x2.65mm_HandSolder, symbol Device:L_Core_Ferrite
- added R1, R2, R3, R6, R7: 10k, Resistor_SMD:R_0603_1608Metric, symbol Device:R
- added R4: 68k, Resistor_SMD:R_0603_1608Metric, symbol Device:R
- added R5: 15k, Resistor_SMD:R_0603_1608Metric, symbol Device:R
- added SW1: SW_Push, Button_Switch_SMD:SW_SPST_CK_RS282G05A3, symbol Switch:SW_Push
- added U2: W25X80, Package_SO:SOIC-8_3.9x4.9mm_P1.27mm, symbol nvitya:W25X80
- added U3: AP3417C, Package_TO_SOT_SMD:SOT-23-5, symbol nvitya:AP3417C
- added Y1: 24MHz, Crystal:Crystal_SMD_3225-4Pin_3.2x2.5mm, symbol Device:Crystal_GND24
- C10: renamed from C5; value 100nF -> 220nF; footprint Capacitor_SMD:C_0603_1608Metric -> Capacitor_SMD:C_0402_1005Metric
- C12: renamed from C6; value 100nF -> 220nF; footprint Capacitor_SMD:C_0603_1608Metric -> Capacitor_SMD:C_0402_1005Metric
- C14: renamed from C7; value 100nF -> 220nF; footprint Capacitor_SMD:C_0603_1608Metric -> Capacitor_SMD:C_0402_1005Metric
- C7: renamed from C14; value 100nF -> 220nF; footprint Capacitor_SMD:C_0603_1608Metric -> Capacitor_SMD:C_0402_1005Metric
- C8: renamed from C4; value 100nF -> 220nF; footprint Capacitor_SMD:C_0603_1608Metric -> Capacitor_SMD:C_0402_1005Metric
- C9: value 22pF -> 4.7uF
- U1: renamed from U?; footprint LQFP100_14X14 -> Package_QFP:LQFP-100_14x14mm_P0.5mm
- renumbered C1 to C2, C2 to C3, R3 to R8, R10 to R9
Connections:
- net labels added: 3V3-EN, A10, A11, A12, A13, A14, A15, A4, A5, A6, A7, A8, A9, B10, B11, B12, B13, B14, B15, BOOT-CFG-0, BOOT-CFG-1, DCDC_OUT, E18, E19, E20, E21, E22, E23, E24, E25, E26, E27, E32, E33, E34, E35, E4, E5, E6, E7, E8, E9, FLASH-CLK, FLASH-CS, FLASH-D0, FLASH-D1, FLASH-D2, FLASH-D3, JTAG-MOD, S0, S1, S2, S3, S4, S5, USB-D+, USB-D-, VDDA
- net labels removed: OSC32_IN, OSC32_OUT
- wire segments 59 -> 281
- no-connect marks 1 -> 8

Commit message: routing finished
Parts:
- removed C1, C22, C25: 220nF, Capacitor_SMD:C_0402_1005Metric, symbol Device:C
- removed C16: 100nF, Capacitor_SMD:C_0603_1608Metric, symbol Device:C
- C17, C23, C24: footprint Capacitor_SMD:C_0603_1608Metric -> Capacitor_SMD:C_0805_2012Metric
- L2, L3: footprint Inductor_SMD:L_1210_3225Metric_Pad1.42x2.65mm_HandSolder -> Inductor_SMD:L_1210_3225Metric
Connections:
- wire segments 281 -> 271
Changed lines of the file:
@@
 F 0 "C17" H 10215 2196 50  0000 L CNN
 F 1 "4.7uF" H 10150 2050 50  0000 L CNN
-F 2 "Capacitor_SMD:C_0603_1608Metric" H 10138 2000 50  0001 C CNN
+F 2 "Capacitor_SMD:C_0805_2012Metric" H 10138 2000 50  0001 C CNN
 F 3 "~" H 10100 2150 50  0001 C CNN
 	1    10100 2150
-	1    0    0    -1
-$EndComp
-$Comp
-L Device:C C16
-U 1 1 5BC2648C
-P 9700 2150
-F 0 "C16" H 9815 2196 50  0000 L CNN
-F 1 "100nF" H 9750 2050 50  0000 L CNN
-F 2 "Capacitor_SMD:C_0603_1608Metric" H 9738 2000 50  0001 C CNN
-F 3 "~" H 9700 2150 50  0001 C CNN
-	1    9700 2150
 	1    0    0    -1
 $EndComp
@@
 F 0 "C24" H 12515 2196 50  0000 L CNN
 F 1 "4.7uF" H 12450 2050 50  0000 L CNN
-F 2 "Capacitor_SMD:C_0603_1608Metric" H 12438 2000 50  0001 C CNN
+F 2 "Capacitor_SMD:C_0805_2012Metric" H 12438 2000 50  0001 C CNN
 F 3 "~" H 12400 2150 50  0001 C CNN
 	1    12400 2150
@@
 Wire Wire Line
 	10100 2600 10100 2300
-Wire Wire Line
-	9700 2300 9700 2600
-Wire Wire Line
-	9700 2600 10100 2600
 Connection ~ 10100 2600
 Wire Wire Line
@@
 Wire Wire Line
 	10100 1800 9700 1800
-Wire Wire Line
-	9700 1800 9700 2000
 Connection ~ 10100 1800
 Wire Wire Line
@@
 Connection ~ 9700 1800
 Wire Wire Line
-	9700 2600 9400 2600
-Connection ~ 9700 2600
-Wire Wire Line
 	12200 2200 10600 2200
 Connection ~ 10600 2200
@@
 F 0 "L2" V 11075 1800 50  0000 C CNN
 F 1 "2.2 uH" V 10984 1800 50  0000 C CNN
-F 2 "Inductor_SMD:L_1210_3225Metric_Pad1.42x2.65mm_HandSolder" H 10850 1800 50  0001 C CNN
+F 2 "Inductor_SMD:L_1210_3225Metric" H 10850 1800 50  0001 C CNN
 F 3 "~" H 10850 1800 50  0001 C CNN
 	1    10850 1800
@@
 F 0 "L3" V 11800 4500 50  0000 C CNN
 F 1 "4.7 uH" V 11900 4500 50  0000 C CNN
-F 2 "Inductor_SMD:L_1210_3225Metric_Pad1.42x2.65mm_HandSolder" H 11950 4500 50  0001 C CNN
+F 2 "Inductor_SMD:L_1210_3225Metric" H 11950 4500 50  0001 C CNN
 F 3 "~" H 11950 4500 50  0001 C CNN
 	1    11950 4500
@@
 F 0 "C23" H 12415 4696 50  0000 L CNN
 F 1 "33uF" H 12350 4550 50  0000 L CNN
-F 2 "Capacitor_SMD:C_0603_1608Metric" H 12338 4500 50  0001 C CNN
+F 2 "Capacitor_SMD:C_0805_2012Metric" H 12338 4500 50  0001 C CNN
 F 3 "~" H 12300 4650 50  0001 C CNN
 	1    12300 4650
@@
 $EndComp
 Wire Wire Line
-	12700 4000 12700 4500
+	12700 4200 12700 4500
 Wire Wire Line
 	11700 5100 11700 5200
@@
 Text Label 13150 3500 2    50   ~ 0
 3V3
-$Comp
-L Device:C C22
-U 1 1 5BCBBC39
-P 12300 4150
-F 0 "C22" H 12300 4250 50  0000 L CNN
-F 1 "220nF" H 12300 4050 50  0000 L CNN
-F 2 "Capacitor_SMD:C_0402_1005Metric" H 12338 4000 50  0001 C CNN
-F 3 "~" H 12300 4150 50  0001 C CNN
-	1    12300 4150
-	1    0    0    -1
-$EndComp
 Wire Wire Line
 	11700 4300 12300 4300
-Wire Wire Line
-	12300 4000 12700 4000
-Wire Wire Line
-	11700 4200 12100 4200
-Wire Wire Line
-	12100 4200 12100 4000
-Wire Wire Line
-	12100 4000 12300 4000
-Connection ~ 12300 4000
-Connection ~ 12300 4300
 $Comp
 L power:GND #PWR0115
@@
 Connection ~ 11850 3400
 $Comp
-L Device:C C25
-U 1 1 5BCE548E
-P 12400 3650
-F 0 "C25" H 12515 3696 50  0000 L CNN
-F 1 "220nF" H 12450 3550 50  0000 L CNN
-F 2 "Capacitor_SMD:C_0402_1005Metric" H 12438 3500 50  0001 C CNN
-F 3 "~" H 12400 3650 50  0001 C CNN
-	1    12400 3650
-	1    0    0    -1
-$EndComp
-$Comp
 L Device:C C28
 U 1 1 5BCE5542
@@
 Wire Wire Line
 	12950 4500 13600 4500
-Wire Wire Line
-	12800 3800 12400 3800
 $Comp
 L power:GND #PWR0116
@@
 	1    0    0    -1
 $EndComp
-Connection ~ 12800 3800
 Wire Wire Line
 	12000 4100 12000 3850
@@
 Wire Wire Line
 	12250 3850 12250 3500
-Wire Wire Line
-	12250 3500 12400 3500
-Connection ~ 12400 3500
-Wire Wire Line
-	12400 3500 12800 3500
 Connection ~ 12800 3500
 Wire Wire Line
@@
 Text Label 6900 2300 0    50   ~ 0
 5V
-$Comp
-L Device:C C1
-U 1 1 5BC39FAB
-P 6000 2550
-F 0 "C1" H 6115 2596 50  0000 L CNN
-F 1 "220nF" H 6050 2450 50  0000 L CNN
-F 2 "Capacitor_SMD:C_0402_1005Metric" H 6038 2400 50  0001 C CNN
-F 3 "~" H 6000 2550 50  0001 C CNN
-	1    6000 2550
-	1    0    0    -1
-$EndComp
 $Comp
 L Device:C C4
@@
 	1    0    0    -1
 $EndComp
-Wire Wire Line
-	6400 2700 6000 2700
 $Comp
 L power:GND #PWR0117
@@
 	1    0    0    -1
 $EndComp
-Connection ~ 6400 2700
-Wire Wire Line
-	6000 2400 6400 2400
 Wire Wire Line
 	7400 2400 6400 2400
-Connection ~ 6400 2400
 NoConn ~ 7400 2700
 Wire Wire Line
@@
 Text Label 6600 4700 2    50   ~ 0
 3V3
+Text Label 1000 8100 0    50   ~ 0
+E4
+Text Label 1000 8000 0    50   ~ 0
+E5
+Text Label 1000 7900 0    50   ~ 0
+E6
+Text Label 1000 7800 0    50   ~ 0
+E7
+Text Label 1000 7600 0    50   ~ 0
+E8
+Text Label 1000 7700 0    50   ~ 0
+E9
+Text Label 1000 7500 0    50   ~ 0
+E18
+Text Label 1000 7400 0    50   ~ 0
+E19
+Text Label 1000 7300 0    50   ~ 0
+E20
+Text Label 1000 7200 0    50   ~ 0
+E21
+Text Label 1000 7100 0    50   ~ 0
+E22
+Text Label 1000 7000 0    50   ~ 0
+E23
+Text Label 1000 6900 0    50   ~ 0
+E24
+Text Label 1000 6800 0    50   ~ 0
+E25
+Text Label 1000 6700 0    50   ~ 0
+E26
+Text Label 1000 6600 0    50   ~ 0
+E27
+Text Label 2800 6600 2    50   ~ 0
+E32
+Text Label 2800 6700 2    50   ~ 0
+E33
+Text Label 2800 6800 2    50   ~ 0
+E34
+Text Label 2800 6900 2    50   ~ 0
+E35
+Text Label 2800 8100 2    50   ~ 0
+B10
+Text Label 2800 8000 2    50   ~ 0
+B11
+Text Label 2800 7900 2    50   ~ 0
+B12
+Text Label 2800 7800 2    50   ~ 0
+B13
+Text Label 2800 7700 2    50   ~ 0
+B14
+Text Label 2800 7600 2    50   ~ 0
+B15
+Text Label 2800 7000 2    50   ~ 0
+A4
+Text Label 2800 7100 2    50   ~ 0
+A5
+Text Label 2800 7200 2    50   ~ 0
+A6
+Text Label 2800 7300 2    50   ~ 0
+A7
+Text Label 2800 7400 2    50   ~ 0
+A8
+Text Label 2800 7500 2    50   ~ 0
+A9
+Text Label 2800 8700 2    50   ~ 0
+A10
+Text Label 2800 8600 2    50   ~ 0
+A11
+Text Label 2800 8500 2    50   ~ 0
+A12
+Text Label 2800 8400 2    50   ~ 0
+A13
+Text Label 2800 8300 2    50   ~ 0
+A14
+Text Label 2800 8200 2    50   ~ 0
+A15
+Text Label 1000 8700 0    50   ~ 0
+S0
 Text Label 1000 8600 0    50   ~ 0
-E4
-Text Label 1000 8700 0    50   ~ 0
-E5
-Text Label 2800 8400 2    50   ~ 0
-E6
-Text Label 2800 8500 2    50   ~ 0
-E7
-Text Label 2800 8600 2    50   ~ 0
-E8
-Text Label 2800 8700 2    50   ~ 0
-E9
-Text Label 1000 6600 0    50   ~ 0
-E18
-Text Label 1000 6700 0    50   ~ 0
-E19
-Text Label 1000 6800 0    50   ~ 0
-E20
-Text Label 1000 6900 0    50   ~ 0
-E21
-Text Label 1000 7000 0    50   ~ 0
-E22
-Text Label 1000 7100 0    50   ~ 0
-E23
-Text Label 1000 7200 0    50   ~ 0
-E24
-Text Label 1000 7300 0    50   ~ 0
-E25
-Text Label 1000 7400 0    50   ~ 0
-E26
-Text Label 1000 7500 0    50   ~ 0
-E27
-Text Label 1000 7600 0    50   ~ 0
-E32
-Text Label 1000 7700 0    50   ~ 0
-E33
-Text Label 1000 7800 0    50   ~ 0
-E34
-Text Label 1000 7900 0    50   ~ 0
-E35
-Text Label 1000 8000 0    50   ~ 0
-B10
-Text Label 1000 8100 0    50   ~ 0
-B11
+S1
+Text Label 1000 8500 0    50   ~ 0
+S2
+Text Label 1000 8400 0    50   ~ 0
+S3
+Text Label 1000 8300 0    50   ~ 0
+S4
 Text Label 1000 8200 0    50   ~ 0
-B12
-Text Label 1000 8300 0    50   ~ 0
-B13
-Text Label 1000 8400 0    50   ~ 0
-B14
-Text Label 1000 8500 0    50   ~ 0
-B15
-Text Label 2800 6600 2    50   ~ 0
-A4
-Text Label 2800 6700 2    50   ~ 0
-A5
-Text Label 2800 6800 2    50   ~ 0
-A6
-Text Label 2800 6900 2    50   ~ 0
-A7
-Text Label 2800 7000 2    50   ~ 0
-A8
-Text Label 2800 7100 2    50   ~ 0
-A9
-Text Label 2800 7200 2    50   ~ 0
-A10
-Text Label 2800 7300 2    50   ~ 0
-A11
-Text Label 2800 7400 2    50   ~ 0
-A12
-Text Label 2800 7500 2    50   ~ 0
-A13
-Text Label 2800 7600 2    50   ~ 0
-A14
-Text Label 2800 7700 2    50   ~ 0
-A15
-Text Label 2800 7800 2    50   ~ 0
-S0
-Text Label 2800 7900 2    50   ~ 0
-S1
-Text Label 2800 8000 2    50   ~ 0
-S2
-Text Label 2800 8100 2    50   ~ 0
-S3
-Text Label 2800 8200 2    50   ~ 0
-S4
-Text Label 2800 8300 2    50   ~ 0
 S5
 Text Label 1000 6400 0    50   ~ 0
@@
 Wire Wire Line
 	6550 1100 7400 1100
+Wire Wire Line
+	9400 2600 10100 2600
+Wire Wire Line
+	12250 3500 12800 3500
+Wire Wire Line
+	11700 4200 12700 4200
 $EndSCHEMATC

Commit message: POR_B and double capacitors
Parts:
- added C1: 22uF, Capacitor_SMD:C_0603_1608Metric, symbol Device:C
- C23: value 33uF -> 22uF; footprint Capacitor_SMD:C_0805_2012Metric -> Capacitor_SMD:C_0603_1608Metric
Connections:
- wire segments 271 -> 275
- no-connect marks 8 -> 7
Changed lines of the file:
@@
 L Device:C C23
 U 1 1 5BC70A9B
-P 12300 4650
-F 0 "C23" H 12415 4696 50  0000 L CNN
-F 1 "33uF" H 12350 4550 50  0000 L CNN
-F 2 "Capacitor_SMD:C_0805_2012Metric" H 12338 4500 50  0001 C CNN
-F 3 "~" H 12300 4650 50  0001 C CNN
-	1    12300 4650
+P 12200 4650
+F 0 "C23" H 12300 4700 50  0000 L CNN
+F 1 "22uF" H 12200 4550 50  0000 L CNN
+F 2 "Capacitor_SMD:C_0603_1608Metric" H 12238 4500 50  0001 C CNN
+F 3 "~" H 12200 4650 50  0001 C CNN
+	1    12200 4650
 	1    0    0    -1
 $EndComp
@@
 L power:GND #PWR0111
 U 1 1 5BC70B70
-P 12300 4800
-F 0 "#PWR0111" H 12300 4550 50  0001 C CNN
-F 1 "GND" H 12305 4627 50  0000 C CNN
-F 2 "" H 12300 4800 50  0001 C CNN
-F 3 "" H 12300 4800 50  0001 C CNN
-	1    12300 4800
+P 12400 4800
+F 0 "#PWR0111" H 12400 4550 50  0001 C CNN
+F 1 "GND" H 12405 4627 50  0000 C CNN
+F 2 "" H 12400 4800 50  0001 C CNN
+F 3 "" H 12400 4800 50  0001 C CNN
+	1    12400 4800
 	1    0    0    -1
 $EndComp
@@
 $EndComp
 Wire Wire Line
-	12300 4500 12100 4500
-Wire Wire Line
-	12700 4500 12300 4500
-Connection ~ 12300 4500
+	12700 4500 12600 4500
 Wire Wire Line
 	12700 4500 12950 4500
@@
 	1    0    0    -1
 $EndComp
-Wire Wire Line
-	9700 6500 9700 6400
 $Comp
 L power:PWR_FLAG #FLG0101
@@
 Wire Wire Line
 	12700 4200 12700 4500
-Wire Wire Line
-	11700 5100 11700 5200
 Text Label 13200 5200 2    50   ~ 0
 DCDC_OUT
@@
 USB-D-
 NoConn ~ 7400 2100
-NoConn ~ 7400 1900
 NoConn ~ 7400 1700
-NoConn ~ 7400 1800
 NoConn ~ 7400 1400
 NoConn ~ 7400 1500
@@
 Wire Wire Line
 	7100 1200 7400 1200
-Connection ~ 9700 3900
-Connection ~ 9700 4000
-Connection ~ 9700 4100
-Connection ~ 9700 4200
-Connection ~ 9700 4300
 $Comp
 L Device:C C6
@@
 Wire Wire Line
 	2400 8900 2800 8900
-Wire Wire Line
-	9700 3900 9700 4000
-Wire Wire Line
-	9700 4000 9700 4100
-Wire Wire Line
-	9700 4100 9700 4200
-Wire Wire Line
-	9700 4200 9700 4300
-Wire Wire Line
-	9700 4300 9700 4400
-Wire Wire Line
-	9700 6400 9700 6300
-Connection ~ 9700 6400
-Connection ~ 9700 5700
-Wire Wire Line
-	9700 5700 9700 5600
-Connection ~ 9700 5800
-Wire Wire Line
-	9700 5800 9700 5700
-Connection ~ 9700 5900
-Wire Wire Line
-	9700 5900 9700 5800
-Connection ~ 9700 6000
-Wire Wire Line
-	9700 6000 9700 5900
-Connection ~ 9700 6100
-Wire Wire Line
-	9700 6100 9700 6000
-Connection ~ 9700 6200
-Wire Wire Line
-	9700 6200 9700 6100
-Connection ~ 9700 6300
-Wire Wire Line
-	9700 6300 9700 6200
-Wire Wire Line
-	11700 4700 11700 4800
-Connection ~ 11700 5100
-Connection ~ 11700 4800
-Wire Wire Line
-	11700 4800 11700 4900
-Connection ~ 11700 4900
-Wire Wire Line
-	11700 4900 11700 5000
-Connection ~ 11700 5000
-Wire Wire Line
-	11700 5000 11700 5100
 $Comp
 L power:PWR_FLAG #FLG0102
@@
 Wire Wire Line
 	11700 4200 12700 4200
+Text Label 6900 1800 0    50   ~ 0
+3V3
+Wire Wire Line
+	9700 3900 9700 4000
+NoConn ~ 7400 1900
+Wire Wire Line
+	7400 1800 6900 1800
+Wire Wire Line
+	11700 5100 11700 5200
+Connection ~ 9700 3900
+Wire Wire Line
+	9700 6400 9700 6500
+Wire Wire Line
+	9700 5600 9700 5700
+Connection ~ 9700 6400
+Connection ~ 9700 5700
+Wire Wire Line
+	9700 5700 9700 5800
+Connection ~ 9700 5800
+Wire Wire Line
+	9700 5800 9700 5900
+Connection ~ 9700 5900
+Wire Wire Line
+	9700 5900 9700 6000
+Connection ~ 9700 6000
+Wire Wire Line
+	9700 6000 9700 6100
+Connection ~ 9700 6100
+Wire Wire Line
+	9700 6100 9700 6200
+Connection ~ 9700 6200
+Wire Wire Line
+	9700 6200 9700 6300
+Connection ~ 9700 6300
+Wire Wire Line
+	9700 6300 9700 6400
+Wire Wire Line
+	11700 5100 11700 5000
+Connection ~ 11700 5100
+Connection ~ 11700 4800
+Wire Wire Line
+	11700 4800 11700 4700
+Connection ~ 11700 4900
+Wire Wire Line
+	11700 4900 11700 4800
+Connection ~ 11700 5000
+Wire Wire Line
+	11700 5000 11700 4900
+Wire Wire Line
+	9700 4400 9700 4300
+Connection ~ 9700 4000
+Connection ~ 9700 4100
+Wire Wire Line
+	9700 4100 9700 4000
+Connection ~ 9700 4200
+Wire Wire Line
+	9700 4200 9700 4100
+Connection ~ 9700 4300
+Wire Wire Line
+	9700 4300 9700 4200
+$Comp
+L Device:C C1
+U 1 1 5BDA6739
+P 12600 4650
+F 0 "C1" H 12715 4696 50  0000 L CNN
+F 1 "22uF" H 12600 4550 50  0000 L CNN
+F 2 "Capacitor_SMD:C_0603_1608Metric" H 12638 4500 50  0001 C CNN
+F 3 "~" H 12600 4650 50  0001 C CNN
+	1    12600 4650
+	1    0    0    -1
+$EndComp
+Connection ~ 12600 4500
+Connection ~ 12200 4500
+Wire Wire Line
+	12200 4500 12600 4500
+Wire Wire Line
+	12100 4500 12200 4500
+Wire Wire Line
+	12600 4800 12400 4800
+Connection ~ 12400 4800
+Wire Wire Line
+	12400 4800 12200 4800
 $EndSCHEMATC
