File: mibo48_xmc4/mibo48_xmc4.kicad_pcb (KiCad board)
At the start: 2 copper layers, 55.9 x 20.3 mm, 32 parts, among them J2 Conn_01x20, J3 Conn_01x20, J4 USB_B_Micro, J5 Conn_01x04, SW1 Reset, U1 XMC4100Q48, U2 AMS1117-3.3, Y1 12MHz, Y2 32.768kHz

Commit message: captioned, gerbers
Parts:
- C11, C8: footprint Capacitor_SMD:C_0603_1608Metric -> Capacitor_SMD:C_1206_3216Metric
- moved C8 1.14 mm to (175.5, 104.9), turned to 0 degrees
- moved C11 0.80 mm to (174.2, 109.0)
- moved U2 0.51 mm to (168.7, 108.0)
Routing:
- net /5V: track 54.4 -> 58.1 mm, vias 3 -> 2
- net +3V3: track 127.0 -> 126.3 mm
- net GND: track 23.5 -> 23.9 mm, vias 23 -> 25
Other:
- board text added: "0.0"
- board text added: "0.1"
- board text added: "0.2"
- board text added: "0.3"
- board text added: "0.4"
- board text added: "0.5"
- board text added: "0.6"
- board text added: "0.7"
- board text added: "0.8"
- board text added: "1.0"
- board text added: "1.1"
- board text added: "1.2"
- board text added: "1.3"
- board text added: "1.4"
- board text added: "1.5"
- board text added: "2.0"
- board text added: "2.1"
- board text added: "2.2"
- board text added: "2.3"
- board text added: "2.4"
- board text added: "2.5"
- board text added: "3V3"
- board text added: "E.0"
- board text added: "E.3"
- board text added: "E.4"
- board text added: "E.5"
- board text added: "E.6"
- board text added: "E.7"
- board text added: "E.8"
- board text added: "E.9"
- board text added: "HIB"
- board text added: "MIBO48-XMC4"
- board text added: "RST"
- board text added: "VDDA"
- board text added: "by nvitya"
- board text removed: "3.3"
