File: mibo48_xmc4/mibo48_xmc4.sch (KiCad schematic (older format))
At the start: 32 parts, among them J2 Conn_01x20, J3 Conn_01x20, J4 USB_B_Micro, J5 Conn_01x04, SW1 Reset, U1 XMC4100Q48, U2 AMS1117-3.3, Y1 12MHz, Y2 32.768kHz

Commit message: captioned, gerbers
Parts:
- C11, C8: footprint Capacitor_SMD:C_0603_1608Metric -> Capacitor_SMD:C_1206_3216Metric
Changed lines of the file:
@@
 F 0 "C8" H 8815 1396 50  0000 L CNN
 F 1 "4.7uF" H 8750 1250 50  0000 L CNN
-F 2 "Capacitor_SMD:C_0603_1608Metric" H 8738 1200 50  0001 C CNN
+F 2 "Capacitor_SMD:C_1206_3216Metric" H 8738 1200 50  0001 C CNN
 F 3 "~" H 8700 1350 50  0001 C CNN
 	1    8700 1350
@@
 F 0 "C11" H 10665 1396 50  0000 L CNN
 F 1 "4.7uF" H 10600 1250 50  0000 L CNN
-F 2 "Capacitor_SMD:C_0603_1608Metric" H 10588 1200 50  0001 C CNN
+F 2 "Capacitor_SMD:C_1206_3216Metric" H 10588 1200 50  0001 C CNN
 F 3 "~" H 10550 1350 50  0001 C CNN
 	1    10550 1350
